File: pcb/goos-right.kicad_sch (KiCad schematic)
At the start: 22 parts

Commit message: fix: switch being permanently on
Connections:
- net at J1.2 (B+), S1.3 (SW): no longer S1.1 (SW)
- no-connect marks 2 -> 3
Changed lines of the file:
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@@
 	(generator_version "8.0")
 	(paper "A4")
-	(junction
-		(at 49.53 74.93)
-		(diameter 0)
-		(color 0 0 0 0)
+	(no_connect
+		(at 49.53 82.55)
 	)
 	(no_connect
@@
 	(wire
 		(pts
-			(xy 69.85 74.93) (xy 49.53 74.93)
-		)
-		(stroke
-			(width 0)
-			(type default)
-		)
-	)
-	(wire
-		(pts
 			(xy 46.99 66.04) (xy 46.99 82.55)
 		)
@@
 	(wire
 		(pts
-			(xy 49.53 74.93) (xy 49.53 82.55)
-		)
-		(stroke
-			(width 0)
-			(type default)
-		)
-	)
-	(wire
-		(pts
-			(xy 44.45 74.93) (xy 49.53 74.93)
+			(xy 44.45 74.93) (xy 69.85 74.93)
 		)
 		(stroke
@@
 		)
 		(instances
-			(project "goos"
+			(project "goos-right"
 				(path "/5166a8b4-1986-48ab-ae39-a65d6d4ad06b"
 					(reference "#PWR019")
@@
 		)
 		(instances
-			(project "goos"
+			(project "goos-right"
 				(path "/5166a8b4-1986-48ab-ae39-a65d6d4ad06b"
 					(reference "#PWR04")
@@
 		)
 		(instances
-			(project "goos"
+			(project "goos-right"
 				(path "/5166a8b4-1986-48ab-ae39-a65d6d4ad06b"
 					(reference "#PWR08")
@@
 		)
 		(instances
-			(project "goos"
+			(project "goos-right"
 				(path "/5166a8b4-1986-48ab-ae39-a65d6d4ad06b"
 					(reference "S2")
@@
 		)
 		(instances
-			(project "goos"
+			(project "goos-right"
 				(path "/5166a8b4-1986-48ab-ae39-a65d6d4ad06b"
 					(reference "#PWR016")
@@
 		)
 		(instances
-			(project "goos"
+			(project "goos-right"
 				(path "/5166a8b4-1986-48ab-ae39-a65d6d4ad06b"
 					(reference "#PWR024")
@@
 		)
 		(instances
-			(project "goos"
+			(project "goos-right"
 				(path "/5166a8b4-1986-48ab-ae39-a65d6d4ad06b"
 					(reference "S19")
@@
 		)
 		(instances
-			(project "goos"
+			(project "goos-right"
 				(path "/5166a8b4-1986-48ab-ae39-a65d6d4ad06b"
 					(reference "#PWR05")
@@
 		)
 		(instances
-			(project "goos"
+			(project "goos-right"
 				(path "/5166a8b4-1986-48ab-ae39-a65d6d4ad06b"
 					(reference "S17")
@@
 		)
 		(instances
-			(project "goos"
+			(project "goos-right"
 				(path "/5166a8b4-1986-48ab-ae39-a65d6d4ad06b"
 					(reference "#PWR014")
@@
 		)
 		(instances
-			(project "goos"
+			(project "goos-right"
 				(path "/5166a8b4-1986-48ab-ae39-a65d6d4ad06b"
 					(reference "#PWR026")
@@
 		)
 		(instances
-			(project "goos"
+			(project "goos-right"
 				(path "/5166a8b4-1986-48ab-ae39-a65d6d4ad06b"
 					(reference "S14")
@@
 		)
 		(instances
-			(project "goos"
+			(project "goos-right"
 				(path "/5166a8b4-1986-48ab-ae39-a65d6d4ad06b"
 					(reference "J1")
@@
 		)
 		(instances
-			(project "goos"
+			(project "goos-right"
 				(path "/5166a8b4-1986-48ab-ae39-a65d6d4ad06b"
 					(reference "S5")
@@
 		)
 		(instances
-			(project "goos"
+			(project "goos-right"
 				(path "/5166a8b4-1986-48ab-ae39-a65d6d4ad06b"
 					(reference "S15")
@@
 		)
 		(instances
-			(project "goos"
+			(project "goos-right"
 				(path "/5166a8b4-1986-48ab-ae39-a65d6d4ad06b"
 					(reference "S13")
@@
 		)
 		(instances
-			(project "goos"
+			(project "goos-right"
 				(path "/5166a8b4-1986-48ab-ae39-a65d6d4ad06b"
 					(reference "#PWR020")
@@
 		)
 		(instances
-			(project "goos"
+			(project "goos-right"
 				(path "/5166a8b4-1986-48ab-ae39-a65d6d4ad06b"
 					(reference "#PWR03")
@@
 		)
 		(instances
-			(project "goos"
+			(project "goos-right"
 				(path "/5166a8b4-1986-48ab-ae39-a65d6d4ad06b"
 					(reference "#PWR021")
@@
 		)
 		(instances
-			(project "goos"
+			(project "goos-right"
 				(path "/5166a8b4-1986-48ab-ae39-a65d6d4ad06b"
 					(reference "JP1")
@@
 		)
 		(instances
-			(project "goos"
+			(project "goos-right"
 				(path "/5166a8b4-1986-48ab-ae39-a65d6d4ad06b"
 					(reference "S4")
@@
 		)
 		(instances
-			(project "goos"
+			(project "goos-right"
 				(path "/5166a8b4-1986-48ab-ae39-a65d6d4ad06b"
 					(reference "S18")
@@
 		)
 		(instances
-			(project "goos"
+			(project "goos-right"
 				(path "/5166a8b4-1986-48ab-ae39-a65d6d4ad06b"
 					(reference "S16")
@@
 		)
 		(instances
-			(project "goos"
+			(project "goos-right"
 				(path "/5166a8b4-1986-48ab-ae39-a65d6d4ad06b"
 					(reference "S11")
@@
 		)
 		(instances
-			(project "goos"
+			(project "goos-right"
 				(path "/5166a8b4-1986-48ab-ae39-a65d6d4ad06b"
 					(reference "S10")
@@
 		)
 		(instances
-			(project "goos"
+			(project "goos-right"
 				(path "/5166a8b4-1986-48ab-ae39-a65d6d4ad06b"
 					(reference "S8")
@@
 		)
 		(instances
-			(project "goos"
+			(project "goos-right"
 				(path "/5166a8b4-1986-48ab-ae39-a65d6d4ad06b"
 					(reference "#PWR025")
@@
 		)
 		(instances
-			(project "goos"
+			(project "goos-right"
 				(path "/5166a8b4-1986-48ab-ae39-a65d6d4ad06b"
 					(reference "S9")
@@
 		)
 		(instances
-			(project "goos"
+			(project "goos-right"
 				(path "/5166a8b4-1986-48ab-ae39-a65d6d4ad06b"
 					(reference "#PWR027")
@@
 		)
 		(instances
-			(project "goos"
+			(project "goos-right"
 				(path "/5166a8b4-1986-48ab-ae39-a65d6d4ad06b"
 					(reference "U1")
@@
 		)
 		(instances
-			(project "goos"
+			(project "goos-right"
 				(path "/5166a8b4-1986-48ab-ae39-a65d6d4ad06b"
 					(reference "S3")
@@
 		)
 		(instances
-			(project "goos"
+			(project "goos-right"
 				(path "/5166a8b4-1986-48ab-ae39-a65d6d4ad06b"
 					(reference "S12")
@@
 		)
 		(instances
-			(project "goos"
+			(project "goos-right"
 				(path "/5166a8b4-1986-48ab-ae39-a65d6d4ad06b"
 					(reference "S1")
@@
 		)
 		(instances
-			(project "goos"
+			(project "goos-right"
 				(path "/5166a8b4-1986-48ab-ae39-a65d6d4ad06b"
 					(reference "#PWR013")
@@
 		)
 		(instances
-			(project "goos"
+			(project "goos-right"
 				(path "/5166a8b4-1986-48ab-ae39-a65d6d4ad06b"
 					(reference "#PWR012")
@@
 		)
 		(instances
-			(project "goos"
+			(project "goos-right"
 				(path "/5166a8b4-1986-48ab-ae39-a65d6d4ad06b"
 					(reference "S6")
@@
 		)
 		(instances
-			(project "goos"
+			(project "goos-right"
 				(path "/5166a8b4-1986-48ab-ae39-a65d6d4ad06b"
 					(reference "#PWR017")
@@
 		)
 		(instances
-			(project "goos"
+			(project "goos-right"
 				(path "/5166a8b4-1986-48ab-ae39-a65d6d4ad06b"
 					(reference "S7")
@@
 		)
 		(instances
-			(project "goos"
+			(project "goos-right"
 				(path "/5166a8b4-1986-48ab-ae39-a65d6d4ad06b"
 					(reference "#PWR011")
@@
 		)
 		(instances
-			(project "goos"
+			(project "goos-right"
 				(path "/5166a8b4-1986-48ab-ae39-a65d6d4ad06b"
 					(reference "#PWR018")
@@
 		)
 		(instances
-			(project "goos"
+			(project "goos-right"
 				(path "/5166a8b4-1986-48ab-ae39-a65d6d4ad06b"
 					(reference "#PWR09")
@@
 		)
 		(instances
-			(project "goos"
+			(project "goos-right"
 				(path "/5166a8b4-1986-48ab-ae39-a65d6d4ad06b"
 					(reference "#PWR07")
@@
 		)
 		(instances
-			(project "goos"
+			(project "goos-right"
 				(path "/5166a8b4-1986-48ab-ae39-a65d6d4ad06b"
 					(reference "#PWR023")
@@
 		)
 		(instances
-			(project "goos"
+			(project "goos-right"
 				(path "/5166a8b4-1986-48ab-ae39-a65d6d4ad06b"
 					(reference "#PWR022")
