File: pcb/goos-left.kicad_pcb (KiCad board)
At the start: 2 copper layers, 142.9 x 112.6 mm, 23 parts

Commit message: feat: added github text
Parts:
- renumbered JP1 to RST
Other:
- board text added: "github.com/FelixBrgm/goos Created by: jgotz && fbruggem V1.0"

Commit message: fix: switch being permanently on
Parts:
- renumbered RST to JP1
Connections:
- S1 pad 3: Net-(J1-B+) -> unconnected-(S1-SW-Pad3)
Routing:
- net Net-(J1-B+): track 68.0 -> 60.1 mm
Changed lines of the file:
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@@
 			(outputformat 1)
 			(mirror no)
-			(drillshape 1)
+			(drillshape 0)
 			(scaleselection 1)
-			(outputdirectory "")
+			(outputdirectory "../../gerbers/")
 		)
 	)
@@
 	(net 24 "unconnected-(U1-VCC-Pad18)")
 	(net 25 "unconnected-(U1-RAW-Pad15)")
+	(net 26 "unconnected-(S1-SW-Pad3)")
 	(footprint "goos:power-switch"
 		(layer "F.Cu")
@@
 			)
 		)
+		(sheetname "Root")
+		(sheetfile "goos-left.kicad_sch")
 		(attr through_hole)
 		(fp_line
@@
 			(size 0.9 1.25)
 			(layers "F.Cu" "F.Paste" "F.Mask")
-			(net 2 "Net-(J1-B+)")
+			(net 26 "unconnected-(S1-SW-Pad3)")
 			(pinfunction "SW")
-			(pintype "passive")
+			(pintype "passive+no_connect")
 		)
 	)
@@
 		)
 		(sheetname "Root")
-		(sheetfile "goos.kicad_sch")
+		(sheetfile "goos-left.kicad_sch")
 		(attr through_hole)
 		(fp_line
@@
 		)
 		(sheetname "Root")
-		(sheetfile "goos.kicad_sch")
+		(sheetfile "goos-left.kicad_sch")
 		(attr through_hole)
 		(fp_line
@@
 		)
 		(sheetname "Root")
-		(sheetfile "goos.kicad_sch")
+		(sheetfile "goos-left.kicad_sch")
 		(attr through_hole)
 		(fp_line
@@
 		)
 		(sheetname "Root")
-		(sheetfile "goos.kicad_sch")
+		(sheetfile "goos-left.kicad_sch")
 		(attr through_hole)
 		(fp_line
@@
 		)
 		(sheetname "Root")
-		(sheetfile "goos.kicad_sch")
+		(sheetfile "goos-left.kicad_sch")
 		(attr through_hole)
 		(fp_line
@@
 		)
 		(sheetname "Root")
-		(sheetfile "goos.kicad_sch")
+		(sheetfile "goos-left.kicad_sch")
 		(attr through_hole)
 		(fp_line
@@
 		(descr "SMD Solder Jumper, 1x1.5mm Triangular Pads, 0.3mm gap, open")
 		(tags "solder jumper open")
-		(property "Reference" "RST"
-			(at 0 -1.8 270)
+		(property "Reference" "JP1"
+			(at 0 -1.8 -90)
 			(layer "F.SilkS")
 			(effects
@@
 		(property ki_fp_filters "SolderJumper*Open*")
 		(sheetname "Root")
-		(sheetfile "goos.kicad_sch")
+		(sheetfile "goos-left.kicad_sch")
 		(zone_connect 1)
 		(attr exclude_from_pos_files)
@@
 		)
 		(sheetname "Root")
-		(sheetfile "goos.kicad_sch")
+		(sheetfile "goos-left.kicad_sch")
 		(attr through_hole)
 		(fp_line
@@
 		)
 		(sheetname "Root")
-		(sheetfile "goos.kicad_sch")
+		(sheetfile "goos-left.kicad_sch")
 		(attr through_hole)
 		(fp_line
@@
 		)
 		(sheetname "Root")
-		(sheetfile "goos.kicad_sch")
+		(sheetfile "goos-left.kicad_sch")
 		(attr through_hole)
 		(fp_line
@@
 		)
 		(sheetname "Root")
-		(sheetfile "goos.kicad_sch")
+		(sheetfile "goos-left.kicad_sch")
 		(attr through_hole)
 		(fp_line
@@
 		)
 		(sheetname "Root")
-		(sheetfile "goos.kicad_sch")
+		(sheetfile "goos-left.kicad_sch")
 		(attr through_hole)
 		(fp_line
@@
 		)
 		(sheetname "Root")
-		(sheetfile "goos.kicad_sch")
+		(sheetfile "goos-left.kicad_sch")
 		(attr through_hole)
 		(fp_line
@@
 		)
 		(sheetname "Root")
-		(sheetfile "goos.kicad_sch")
+		(sheetfile "goos-left.kicad_sch")
 		(attr through_hole)
 		(fp_line
@@
 		)
 		(sheetname "Root")
-		(sheetfile "goos.kicad_sch")
+		(sheetfile "goos-left.kicad_sch")
 		(attr through_hole)
 		(fp_line
@@
 		)
 		(sheetname "Root")
-		(sheetfile "goos.kicad_sch")
+		(sheetfile "goos-left.kicad_sch")
 		(attr through_hole)
 		(fp_line
@@
 		)
 		(sheetname "Root")
-		(sheetfile "goos.kicad_sch")
+		(sheetfile "goos-left.kicad_sch")
 		(attr through_hole)
 		(fp_line
@@
 		)
 		(sheetname "Root")
-		(sheetfile "goos.kicad_sch")
+		(sheetfile "goos-left.kicad_sch")
 		(attr through_hole)
 		(fp_line
@@
 		)
 		(sheetname "Root")
-		(sheetfile "goos.kicad_sch")
+		(sheetfile "goos-left.kicad_sch")
 		(attr through_hole)
 		(fp_line
@@
 		)
 		(sheetname "Root")
-		(sheetfile "goos.kicad_sch")
+		(sheetfile "goos-left.kicad_sch")
 		(attr through_hole)
 		(fp_line
@@
 		)
 		(sheetname "Root")
-		(sheetfile "goos.kicad_sch")
+		(sheetfile "goos-left.kicad_sch")
 		(attr through_hole)
 		(fp_text user "B+"
@@
 	)
 	(segment
-		(start 74.5 104.422949)
-		(end 74.5 101.066783)
-		(width 0.2)
-		(layer "F.Cu")
-		(net 2)
-	)
-	(segment
 		(start 78.149998 85.149998)
 		(end 77.270706 84.270706)
@@
 		(net 2)
 	)
-	(segment
-		(start 74.661229 100.905554)
-		(end 76.46521 100.905554)
-		(width 0.2)
-		(layer "F.Cu")
-		(net 2)
-	)
-	(segment
-		(start 75.482605 105.405554)
-		(end 76.46521 105.405554)
-		(width 0.2)
-		(layer "F.Cu")
-		(net 2)
-	)
 	(via
 		(at 77.199997 84)
@@
 	)
 	(arc
-		(start 74.5 104.422949)
-		(mid 74.787798 105.117755)
-		(end 75.482605 105.405554)
-		(width 0.2)
-		(layer "F.Cu")
-		(net 2)
-	)
-	(arc
-		(start 74.547223 100.952777)
-		(mid 74.512272 101.005083)
-		(end 74.5 101.066783)
-		(width 0.2)
-		(layer "F.Cu")
-		(net 2)
-	)
-	(arc
 		(start 79.1 99.188965)
 		(mid 78.969332 99.845875)
@@
 		(width 0.2)
 		(layer "F.Cu")
-		(net 2)
-	)
-	(arc
-		(start 74.661229 100.905554)
-		(mid 74.599529 100.917826)
-		(end 74.547223 100.952777)
-		(width 0.2)
-		(layer "F.Cu")

Commit message: feat: fixed right half
Parts:
- removed ?: , 
- renumbered JP1 to RST
Other:
- board text added: "github.com/FelixBrgm/goos Created by: jgotz && fbruggem V0.0.1"
- board text removed: "github.com/FelixBrgm/goos Created by: jgotz && fbruggem V1.0"
