File: pcb/goos-left.kicad_pcb (KiCad board)
At the start: 2 copper layers, 142.9 x 112.6 mm, 22 parts

Commit message: fix: move pads further apart
Routing:
- net Net-(J1-B+): track 60.1 -> 59.1 mm
Other:
- board text added: "github.com/FelixBrgm/goos Created by: jgotz && fbruggem V0.0.2"
- board text removed: "github.com/FelixBrgm/goos Created by: jgotz && fbruggem V0.0.1"
